Commit message: decrease_robot_size

File: urdf/spcbot/spcbot.gazebo.xacro (robot description, xacro)
@@ -5,5 +5,5 @@
     <sensor type="camera" name="camera">
       <update_rate>30.0</update_rate>
-      <visualize>true</visualize>
+      <visualize></visualize>
       <camera name="head">
         <horizontal_fov>1.3962634</horizontal_fov>
@@ -73,5 +73,5 @@
   <gazebo reference="hokuyo_link">
     <sensor type="ray" name="head_hokuyo_sensor">
-      <pose>0.15 0 0.1 0 0 0</pose>
+      <pose>0.075 0 0.05 0 0 0</pose>
       <visualize>ture</visualize>
       <update_rate>40</update_rate>

File: urdf/spcbot/spcbot.urdf.xacro (robot description, xacro)
@@ -1,5 +1,5 @@
 <?xml version='1.0'?>
 <robot name="myrobot" xmlns:xacro="http://www.ros.org/wiki/xacro">
-  <xacro:property name="cameraSize" value="0.05"/>
+  <xacro:property name="cameraSize" value="0.025"/>
   <xacro:property name="cameraMass" value="0.1"/>
   <!-- <xacro:include filename="$(find spcbot_description)/urdf/materials.xacro"/> -->
@@ -18,5 +18,5 @@
     <collision name='collision'>
       <geometry>
-        <box size=".4 .2 .1"/>
+        <box size=".15 .1 .05"/>
       </geometry>
     </collision>
@@ -24,12 +24,12 @@
       <origin xyz="0 0 0" rpy=" 0 0 0"/>
       <geometry>
-        <box size=".4 .2 .1"/>
+        <box size=".15 .1 .05"/>
       </geometry>
       <material name="black"/>
     </visual>
     <collision name='caster_collision'>
-      <origin xyz="-0.15 0 -0.05" rpy=" 0 0 0"/>
+      <origin xyz="-0.055 0 -0.025" rpy=" 0 0 0"/>
       <geometry>
-        <sphere radius="0.05"/>
+        <sphere radius="0.025"/>
       </geometry>
       <!-- <surface>
@@ -45,15 +45,15 @@
     </collision>
     <visual name='caster_visual'>
-      <origin xyz="-0.15 0 -0.05" rpy=" 0 0 0"/>
+      <origin xyz="-0.055 0 -0.025" rpy=" 0 0 0"/>
       <geometry>
-        <sphere radius="0.05"/>
+        <sphere radius="0.025"/>
       </geometry>
     </visual>
-    <collision name='caster_front_collision'>
-      <origin xyz="0.15 0 -0.05" rpy=" 0 0 0"/>
+    <!-- <collision name='caster_front_collision'>
+      <origin xyz="0.075 0 -0.025" rpy=" 0 0 0"/>
       <geometry>
-        <sphere radius="0.05"/>
+        <sphere radius="0.025"/>
       </geometry>
-      <!-- <surface>
+      < <surface>
         <friction>
           <ode>
@@ -64,12 +64,12 @@
           </ode>
         </friction>
-      </surface> -->
+      </surface> >
     </collision>
     <visual name='caster_front_visual'>
-      <origin xyz="0.15 0 -0.05" rpy=" 0 0 0"/>
+      <origin xyz="0.075 0 -0.025" rpy=" 0 0 0"/>
       <geometry>
-        <sphere radius="0.05"/>
+        <sphere radius="0.025"/>
       </geometry>
-    </visual>
+    </visual> -->
   </link>
   <link name="left_wheel">
@@ -78,5 +78,5 @@
       <origin xyz="0 0 0" rpy="0 1.5707 1.5707"/>
       <geometry>
-        <cylinder radius="0.1" length="0.05"/>
+        <cylinder radius="0.05" length="0.025"/>
       </geometry>
     </collision>
@@ -84,5 +84,5 @@
       <origin xyz="0 0 0" rpy="0 1.5707 1.5707"/>
       <geometry>
-        <cylinder radius="0.1" length="0.05"/>
+        <cylinder radius="0.05" length="0.025"/>
       </geometry>
       <material name="yellow"/>
@@ -102,5 +102,5 @@
       <origin xyz="0 0 0" rpy="0 1.5707 1.5707"/>
       <geometry>
-        <cylinder radius="0.1" length="0.05"/>
+        <cylinder radius="0.05" length="0.025"/>
       </geometry>
     </collision>
@@ -108,5 +108,5 @@
       <origin xyz="0 0 0" rpy="0 1.5707 1.5707"/>
       <geometry>
-        <cylinder radius="0.1" length="0.05"/>
+        <cylinder radius="0.05" length="0.025"/>
       </geometry>
       <material name="yellow"/>
@@ -122,5 +122,5 @@
   </link>
   <joint type="continuous" name="left_wheel_hinge">
-    <origin xyz="0 0.15 0" rpy="0 0 0"/>
+    <origin xyz=".055 0.075 0" rpy="0 0 0"/>
     <!--origin xyz="0.1 0.13 0" rpy="0 1.5707 1.5707"/-->
     <child link="left_wheel"/>
@@ -131,5 +131,5 @@
   </joint>
   <joint type="continuous" name="right_wheel_hinge">
-    <origin xyz="0 -0.15 0" rpy="0 0 0"/>
+    <origin xyz=".055 -0.075 0" rpy="0 0 0"/>
     <!--origin xyz="0.1 -0.13 0" rpy="0 1.5707 1.5707"/-->
     <child link="right_wheel"/>
@@ -162,5 +162,5 @@
   <joint name="camera_joint" type="fixed">
     <axis xyz="0 1 0" />
-    <origin xyz=".2 0 0" rpy="0 0 0"/>
+    <origin xyz=".075 0 0" rpy="0 0 0"/>
     <parent link="chassis"/>
     <child link="camera_link"/>
