Commit message: perfect_move

File: urdf/camera.xacro (robot description, xacro)
@@ -6,5 +6,5 @@
       <visual>
         <geometry>
-          <mesh filename="package://computer_vision_pkg/meshes/head.dae" scale=".5 .5 .5"/>
+          <mesh filename="package://cv/meshes/head.dae" scale=".5 .5 .5"/>
         </geometry>
       </visual>

File: urdf/spcbot/spcbot.urdf.xacro (robot description, xacro)
@@ -4,5 +4,5 @@
   <xacro:property name="cameraMass" value="0.1"/>
   <!-- <xacro:include filename="$(find spcbot_description)/urdf/materials.xacro"/> -->
-  <xacro:include filename="$(find computer_vision_pkg)/urdf/spcbot/spcbot.gazebo.xacro"/>
+  <xacro:include filename="$(find cv)/urdf/spcbot/spcbot.gazebo.xacro"/>
   <link name='chassis'>
     <pose>0 0 0.1 0 0 0</pose>
@@ -29,7 +29,7 @@
     </visual>
     <collision name='caster_collision'>
-      <origin xyz="-0.055 0 -0.025" rpy=" 0 0 0"/>
+      <origin xyz="-0.055 0 -0.02" rpy=" 0 0 0"/>
       <geometry>
-        <sphere radius="0.025"/>
+        <sphere radius="0.02"/>
       </geometry>
       <!-- <surface>
@@ -45,7 +45,7 @@
     </collision>
     <visual name='caster_visual'>
-      <origin xyz="-0.055 0 -0.025" rpy=" 0 0 0"/>
+      <origin xyz="-0.055 0 -0.02" rpy=" 0 0 0"/>
       <geometry>
-        <sphere radius="0.025"/>
+        <sphere radius="0.02"/>
       </geometry>
     </visual>
@@ -78,5 +78,5 @@
       <origin xyz="0 0 0" rpy="0 1.5707 1.5707"/>
       <geometry>
-        <cylinder radius="0.05" length="0.025"/>
+        <cylinder radius="0.04" length="0.02"/>
       </geometry>
     </collision>
@@ -84,5 +84,5 @@
       <origin xyz="0 0 0" rpy="0 1.5707 1.5707"/>
       <geometry>
-        <cylinder radius="0.05" length="0.025"/>
+        <cylinder radius="0.04" length="0.02"/>
       </geometry>
       <material name="yellow"/>
@@ -102,5 +102,5 @@
       <origin xyz="0 0 0" rpy="0 1.5707 1.5707"/>
       <geometry>
-        <cylinder radius="0.05" length="0.025"/>
+        <cylinder radius="0.04" length="0.02"/>
       </geometry>
     </collision>
@@ -108,5 +108,5 @@
       <origin xyz="0 0 0" rpy="0 1.5707 1.5707"/>
       <geometry>
-        <cylinder radius="0.05" length="0.025"/>
+        <cylinder radius="0.04" length="0.02"/>
       </geometry>
       <material name="yellow"/>
@@ -122,5 +122,5 @@
   </link>
   <joint type="continuous" name="left_wheel_hinge">
-    <origin xyz=".055 0.075 0" rpy="0 0 0"/>
+    <origin xyz=".045 0.075 0" rpy="0 0 0"/>
     <!--origin xyz="0.1 0.13 0" rpy="0 1.5707 1.5707"/-->
     <child link="left_wheel"/>
@@ -131,5 +131,5 @@
   </joint>
   <joint type="continuous" name="right_wheel_hinge">
-    <origin xyz=".055 -0.075 0" rpy="0 0 0"/>
+    <origin xyz=".045 -0.075 0" rpy="0 0 0"/>
     <!--origin xyz="0.1 -0.13 0" rpy="0 1.5707 1.5707"/-->
     <child link="right_wheel"/>

File: urdf/sumo.urdf.xacro (robot description, xacro)
@@ -1,6 +1,6 @@
 <?xml version="1.0"?>
 <robot xmlns:xacro="http://www.ros.org/wiki/xacro" name="sumo">
-  <xacro:include filename="$(find computer_vision_pkg)/urdf/wheel.xacro" />
-  <xacro:include filename="$(find computer_vision_pkg)/urdf/camera.xacro" />
+  <xacro:include filename="$(find cv)/urdf/wheel.xacro" />
+  <xacro:include filename="$(find cv)/urdf/camera.xacro" />
   <xacro:property name="base_length" value=".15" />
   <link name="base_link">
